Commit message: missed a few sr_mst refs

File: sr_description/hand/xacro/finger/distal/f_distal_mst.urdf.xacro (robot description, xacro)
@@ -32,5 +32,5 @@
                 <origin xyz="0 0 0" rpy="0 0 0"/>
                 <geometry>
-                    <mesh filename="package://sr_mst/meshes/f_distal/f_distal_mst.dae" scale="${scale} ${scale} ${scale}"/>
+                    <mesh filename="package://sr_description/meshes/components/f_distal/mst/f_distal_mst.dae" scale="${scale} ${scale} ${scale}"/>
                 </geometry>
             </visual>
@@ -38,5 +38,5 @@
                 <origin xyz="0 0 0" rpy="0 0 0"/>
                 <geometry>
-                    <mesh filename="package://sr_mst/meshes/f_distal/f_distal_mst.dae" scale="${scale} ${scale} ${scale}"/>
+                    <mesh filename="package://sr_description/meshes/components/f_distal/mst/f_distal_mst.dae" scale="${scale} ${scale} ${scale}"/>
                 </geometry>
             </collision>

File: sr_description/hand/xacro/finger/distal/f_distal_mstXL.urdf.xacro (robot description, xacro)
@@ -32,5 +32,5 @@
                 <origin xyz="0 0 0" rpy="0 0 0"/>
                 <geometry>
-                    <mesh filename="package://sr_mst/meshes/f_distal_XL/f_distal_mstXL.dae" scale="${scale} ${scale} ${scale}"/>
+                    <mesh filename="package://sr_description/meshes/components/f_distal/mst/f_distal_mstXL.dae" scale="${scale} ${scale} ${scale}"/>
                 </geometry>
             </visual>
@@ -38,5 +38,5 @@
                 <origin xyz="0 0 0" rpy="0 0 0"/>
                 <geometry>
-                    <mesh filename="package://sr_mst/meshes/f_distal_XL/f_distal_mstXL.dae" scale="${scale} ${scale} ${scale}"/>
+                    <mesh filename="package://sr_description/meshes/components/f_distal/mst/f_distal_mstXL.dae" scale="${scale} ${scale} ${scale}"/>
                 </geometry>
             </collision>

File: sr_description/hand/xacro/thumb/th_distal_mst.urdf.xacro (robot description, xacro)
@@ -32,5 +32,5 @@
                 <origin xyz="0 0 0" rpy="0 0 0"/>
                 <geometry>
-                    <mesh filename="package://sr_mst/meshes/th_distal/th_distal_mst.dae" scale="${scale} ${scale} ${scale}"/>
+                    <mesh filename="package://sr_description/meshes/components/th_distal/mst/th_distal_mst.dae" scale="${scale} ${scale} ${scale}"/>
                 </geometry>
             </visual>
@@ -38,5 +38,5 @@
                 <origin xyz="0 0 0" rpy="0 0 0"/>
                 <geometry>
-                    <mesh filename="package://sr_mst/meshes/th_distal/th_distal_mst.dae" scale="${scale} ${scale} ${scale}"/>
+                    <mesh filename="package://sr_description/meshes/components/th_distal/mst/th_distal_mst.dae" scale="${scale} ${scale} ${scale}"/>
                 </geometry>
             </collision>
