Commit message: Fix identation

File: sr_description/hand/xacro/finger/distal/distal.urdf.xacro (robot description, xacro)
@@ -41,44 +41,44 @@
         <inertia ixx="0.00000094" ixy="0.0" ixz="0.0" iyy="0.0000011" iyz="0.0" izz="0.00000053" />
       </inertial>
-        <visual>
-          <origin xyz="0 0 0" rpy="0 0 0" />
-          <geometry name="${prefix}${link_prefix}distal_visual">
-            <xacro:if value="${tip_sensor == 'pst'}">
-              <mesh filename="package://sr_description/meshes/components/f_distal/pst/f_distal_pst.dae"
-                    scale="0.001 0.001 0.001" />
-            </xacro:if>
-            <xacro:if value="${tip_sensor == 'bt_sp'}">
-              <mesh filename="package://sr_description/meshes/components/f_distal/bt_sp/f_distal_bt_sp.dae"
-                    scale="0.001 0.001 0.001" />
-            </xacro:if>
-            <xacro:if value="${tip_sensor == 'bt_2p'}">
-              <mesh filename="package://sr_description/meshes/components/f_distal/bt_2p/f_distal_bt_2p.dae" />
-            </xacro:if>
-            <xacro:if value="${tip_sensor == 'mst'}">
-              <mesh filename="package://sr_mst/meshes/f_distal_XL/f_distal_mstXL.dae"
+      <visual>
+        <origin xyz="0 0 0" rpy="0 0 0" />
+        <geometry name="${prefix}${link_prefix}distal_visual">
+          <xacro:if value="${tip_sensor == 'pst'}">
+            <mesh filename="package://sr_description/meshes/components/f_distal/pst/f_distal_pst.dae"
                   scale="0.001 0.001 0.001" />
-            </xacro:if>
-          </geometry>
-        </visual>
-        <collision>
-          <origin xyz="0 0 0" rpy="0 0 0" />
-          <geometry name="${prefix}${link_prefix}distal_collision_geom">
-            <xacro:if value="${tip_sensor == 'pst'}">
-              <mesh filename="package://sr_description/meshes/components/f_distal/pst/f_distal_pst.dae"
-                    scale="0.001 0.001 0.001" />
-            </xacro:if>
-            <xacro:if value="${tip_sensor == 'bt_sp'}">
-              <mesh filename="package://sr_description/meshes/components/f_distal/bt_sp/f_distal_bt_sp.dae"
-                    scale="0.001 0.001 0.001" />
-            </xacro:if>
-            <xacro:if value="${tip_sensor == 'bt_2p'}">
-              <mesh filename="package://sr_description/meshes/components/f_distal/bt_2p/f_distal_bt_2p.dae" />
-            </xacro:if>
-            <xacro:if value="${tip_sensor == 'mst'}">
-              <mesh filename="package://sr_mst/meshes/f_distal_XL/f_distal_mstXL.dae"
+          </xacro:if>
+          <xacro:if value="${tip_sensor == 'bt_sp'}">
+            <mesh filename="package://sr_description/meshes/components/f_distal/bt_sp/f_distal_bt_sp.dae"
                   scale="0.001 0.001 0.001" />
-            </xacro:if>
-          </geometry>
-        </collision>
+          </xacro:if>
+          <xacro:if value="${tip_sensor == 'bt_2p'}">
+            <mesh filename="package://sr_description/meshes/components/f_distal/bt_2p/f_distal_bt_2p.dae" />
+          </xacro:if>
+          <xacro:if value="${tip_sensor == 'mst'}">
+            <mesh filename="package://sr_mst/meshes/f_distal_XL/f_distal_mstXL.dae"
+                scale="0.001 0.001 0.001" />
+          </xacro:if>
+        </geometry>
+      </visual>
+      <collision>
+        <origin xyz="0 0 0" rpy="0 0 0" />
+        <geometry name="${prefix}${link_prefix}distal_collision_geom">
+          <xacro:if value="${tip_sensor == 'pst'}">
+            <mesh filename="package://sr_description/meshes/components/f_distal/pst/f_distal_pst.dae"
+                  scale="0.001 0.001 0.001" />
+          </xacro:if>
+          <xacro:if value="${tip_sensor == 'bt_sp'}">
+            <mesh filename="package://sr_description/meshes/components/f_distal/bt_sp/f_distal_bt_sp.dae"
+                  scale="0.001 0.001 0.001" />
+          </xacro:if>
+          <xacro:if value="${tip_sensor == 'bt_2p'}">
+            <mesh filename="package://sr_description/meshes/components/f_distal/bt_2p/f_distal_bt_2p.dae" />
+          </xacro:if>
+          <xacro:if value="${tip_sensor == 'mst'}">
+            <mesh filename="package://sr_mst/meshes/f_distal_XL/f_distal_mstXL.dae"
+                scale="0.001 0.001 0.001" />
+          </xacro:if>
+        </geometry>
+      </collision>
     </link>
     <xacro:unless value="${tip_sensor == 'bt_2p'}">

Commit message: adding mst xacros, meshes

File: sr_description/hand/xacro/finger/distal/distal.urdf.xacro (robot description, xacro)
@@ -33,5 +33,5 @@
   <xacro:include filename="$(find sr_description)/hand/xacro/finger/distal/distal.gazebo.xacro" />
   <xacro:include filename="$(find sr_description)/hand/xacro/finger/distal/distal.transmission.xacro" />
-  <xacro:include filename="$(find sr_mst)/xacro/f_distalXL.urdf.xacro" />
+  <xacro:include filename="$(find sr_description)/hand/xacro/finger/distal/f_distal_mstXL.urdf.xacro" />
   <xacro:macro name="distal" params="prefix:=^ link_prefix:=^ joint_prefix:=^ tip_sensor:=^|pst parent">
     <link name="${prefix}${link_prefix}distal">
@@ -56,5 +56,5 @@
             </xacro:if>
             <xacro:if value="${tip_sensor == 'mst'}">
-              <mesh filename="package://sr_mst/meshes/f_distal_XL/f_distal_mstXL.dae"
+              <mesh filename="package://sr_description/meshes/components/f_distal/mst/f_distal_mstXL.dae"
                   scale="0.001 0.001 0.001" />
             </xacro:if>
@@ -76,5 +76,5 @@
             </xacro:if>
             <xacro:if value="${tip_sensor == 'mst'}">
-              <mesh filename="package://sr_mst/meshes/f_distal_XL/f_distal_mstXL.dae"
+              <mesh filename="package://sr_description/meshes/components/f_distal/mst/f_distal_mstXL.dae"
                   scale="0.001 0.001 0.001" />
             </xacro:if>

File: sr_description/hand/xacro/thumb/thdistal.urdf.xacro (robot description, xacro)
@@ -33,5 +33,5 @@
   <xacro:include filename="$(find sr_description)/hand/xacro/thumb/thdistal.gazebo.xacro" />
   <xacro:include filename="$(find sr_description)/hand/xacro/thumb/thdistal.transmission.xacro" />
-  <xacro:include filename="$(find sr_mst)/xacro/th_distal.urdf.xacro" />
+  <xacro:include filename="$(find sr_description)/hand/xacro/thumb/th_distal_mst.urdf.xacro" />
   <xacro:macro name="thdistal" params="tip_sensor:=^|pst prefix:=^ parent">
     <xacro:if value="${tip_sensor == 'bt_2p'}">
@@ -134,5 +134,5 @@
             </xacro:if>
             <xacro:if value="${tip_sensor == 'mst'}">
-              <mesh filename="package://sr_mst/meshes/th_distal/th_distal_mst.dae"
+              <mesh filename="package://sr_description/meshes/components/th_distal/mst/th_distal_mst.dae"
                     scale="0.001 0.001 0.001" />
             </xacro:if>
@@ -158,5 +158,5 @@
             </xacro:if>
             <xacro:if value="${tip_sensor == 'mst'}">
-              <mesh filename="package://sr_mst/meshes/th_distal/th_distal_mst.dae"
+              <mesh filename="package://sr_description/meshes/components/th_distal/mst/th_distal_mst.dae"
                     scale="0.001 0.001 0.001" />
             </xacro:if>

Commit message: undo formatting commit

File: sr_description/hand/xacro/finger/distal/distal.urdf.xacro (robot description, xacro)
@@ -2,5 +2,5 @@
 <!--
  Software License Agreement (BSD License)
- Copyright © 2022-2024 belongs to Shadow Robot Company Ltd.
+ Copyright © 2022-2023 belongs to Shadow Robot Company Ltd.
  All rights reserved.
  Redistribution and use in source and binary forms, with or without modification,
@@ -41,44 +41,44 @@
         <inertia ixx="0.00000094" ixy="0.0" ixz="0.0" iyy="0.0000011" iyz="0.0" izz="0.00000053" />
       </inertial>
-      <visual>
-        <origin xyz="0 0 0" rpy="0 0 0" />
-        <geometry name="${prefix}${link_prefix}distal_visual">
-          <xacro:if value="${tip_sensor == 'pst'}">
-            <mesh filename="package://sr_description/meshes/components/f_distal/pst/f_distal_pst.dae"
+        <visual>
+          <origin xyz="0 0 0" rpy="0 0 0" />
+          <geometry name="${prefix}${link_prefix}distal_visual">
+            <xacro:if value="${tip_sensor == 'pst'}">
+              <mesh filename="package://sr_description/meshes/components/f_distal/pst/f_distal_pst.dae"
+                    scale="0.001 0.001 0.001" />
+            </xacro:if>
+            <xacro:if value="${tip_sensor == 'bt_sp'}">
+              <mesh filename="package://sr_description/meshes/components/f_distal/bt_sp/f_distal_bt_sp.dae"
+                    scale="0.001 0.001 0.001" />
+            </xacro:if>
+            <xacro:if value="${tip_sensor == 'bt_2p'}">
+              <mesh filename="package://sr_description/meshes/components/f_distal/bt_2p/f_distal_bt_2p.dae" />
+            </xacro:if>
+            <xacro:if value="${tip_sensor == 'mst'}">
+              <mesh filename="package://sr_mst/meshes/f_distal_XL/f_distal_mstXL.dae"
                   scale="0.001 0.001 0.001" />
-          </xacro:if>
-          <xacro:if value="${tip_sensor == 'bt_sp'}">
-            <mesh filename="package://sr_description/meshes/components/f_distal/bt_sp/f_distal_bt_sp.dae"
+            </xacro:if>
+          </geometry>
+        </visual>
+        <collision>
+          <origin xyz="0 0 0" rpy="0 0 0" />
+          <geometry name="${prefix}${link_prefix}distal_collision_geom">
+            <xacro:if value="${tip_sensor == 'pst'}">
+              <mesh filename="package://sr_description/meshes/components/f_distal/pst/f_distal_pst.dae"
+                    scale="0.001 0.001 0.001" />
+            </xacro:if>
+            <xacro:if value="${tip_sensor == 'bt_sp'}">
+              <mesh filename="package://sr_description/meshes/components/f_distal/bt_sp/f_distal_bt_sp.dae"
+                    scale="0.001 0.001 0.001" />
+            </xacro:if>
+            <xacro:if value="${tip_sensor == 'bt_2p'}">
+              <mesh filename="package://sr_description/meshes/components/f_distal/bt_2p/f_distal_bt_2p.dae" />
+            </xacro:if>
+            <xacro:if value="${tip_sensor == 'mst'}">
+              <mesh filename="package://sr_mst/meshes/f_distal_XL/f_distal_mstXL.dae"
                   scale="0.001 0.001 0.001" />
-          </xacro:if>
-          <xacro:if value="${tip_sensor == 'bt_2p'}">
-            <mesh filename="package://sr_description/meshes/components/f_distal/bt_2p/f_distal_bt_2p.dae" />
-          </xacro:if>
-          <xacro:if value="${tip_sensor == 'mst'}">
-            <mesh filename="package://sr_mst/meshes/f_distal_XL/f_distal_mstXL.dae"
-                scale="0.001 0.001 0.001" />
-          </xacro:if>
-        </geometry>
-      </visual>
-      <collision>
-        <origin xyz="0 0 0" rpy="0 0 0" />
-        <geometry name="${prefix}${link_prefix}distal_collision_geom">
-          <xacro:if value="${tip_sensor == 'pst'}">
-            <mesh filename="package://sr_description/meshes/components/f_distal/pst/f_distal_pst.dae"
-                  scale="0.001 0.001 0.001" />
-          </xacro:if>
-          <xacro:if value="${tip_sensor == 'bt_sp'}">
-            <mesh filename="package://sr_description/meshes/components/f_distal/bt_sp/f_distal_bt_sp.dae"
-                  scale="0.001 0.001 0.001" />
-          </xacro:if>
-          <xacro:if value="${tip_sensor == 'bt_2p'}">
-            <mesh filename="package://sr_description/meshes/components/f_distal/bt_2p/f_distal_bt_2p.dae" />
-          </xacro:if>
-          <xacro:if value="${tip_sensor == 'mst'}">
-            <mesh filename="package://sr_mst/meshes/f_distal_XL/f_distal_mstXL.dae"
-                scale="0.001 0.001 0.001" />
-          </xacro:if>
-        </geometry>
-      </collision>
+            </xacro:if>
+          </geometry>
+        </collision>
     </link>
     <xacro:unless value="${tip_sensor == 'bt_2p'}">

Commit message: formatting

File: sr_description/hand/xacro/finger/distal/distal.urdf.xacro (robot description, xacro)
@@ -41,44 +41,44 @@
         <inertia ixx="0.00000094" ixy="0.0" ixz="0.0" iyy="0.0000011" iyz="0.0" izz="0.00000053" />
       </inertial>
-        <visual>
-          <origin xyz="0 0 0" rpy="0 0 0" />
-          <geometry name="${prefix}${link_prefix}distal_visual">
-            <xacro:if value="${tip_sensor == 'pst'}">
-              <mesh filename="package://sr_description/meshes/components/f_distal/pst/f_distal_pst.dae"
-                    scale="0.001 0.001 0.001" />
-            </xacro:if>
-            <xacro:if value="${tip_sensor == 'bt_sp'}">
-              <mesh filename="package://sr_description/meshes/components/f_distal/bt_sp/f_distal_bt_sp.dae"
-                    scale="0.001 0.001 0.001" />
-            </xacro:if>
-            <xacro:if value="${tip_sensor == 'bt_2p'}">
-              <mesh filename="package://sr_description/meshes/components/f_distal/bt_2p/f_distal_bt_2p.dae" />
-            </xacro:if>
-            <xacro:if value="${tip_sensor == 'mst'}">
-              <mesh filename="package://sr_description/meshes/components/f_distal/mst/f_distal_mstXL.dae"
+      <visual>
+        <origin xyz="0 0 0" rpy="0 0 0" />
+        <geometry name="${prefix}${link_prefix}distal_visual">
+          <xacro:if value="${tip_sensor == 'pst'}">
+            <mesh filename="package://sr_description/meshes/components/f_distal/pst/f_distal_pst.dae"
                   scale="0.001 0.001 0.001" />
-            </xacro:if>
-          </geometry>
-        </visual>
-        <collision>
-          <origin xyz="0 0 0" rpy="0 0 0" />
-          <geometry name="${prefix}${link_prefix}distal_collision_geom">
-            <xacro:if value="${tip_sensor == 'pst'}">
-              <mesh filename="package://sr_description/meshes/components/f_distal/pst/f_distal_pst.dae"
-                    scale="0.001 0.001 0.001" />
-            </xacro:if>
-            <xacro:if value="${tip_sensor == 'bt_sp'}">
-              <mesh filename="package://sr_description/meshes/components/f_distal/bt_sp/f_distal_bt_sp.dae"
-                    scale="0.001 0.001 0.001" />
-            </xacro:if>
-            <xacro:if value="${tip_sensor == 'bt_2p'}">
-              <mesh filename="package://sr_description/meshes/components/f_distal/bt_2p/f_distal_bt_2p.dae" />
-            </xacro:if>
-            <xacro:if value="${tip_sensor == 'mst'}">
-              <mesh filename="package://sr_description/meshes/components/f_distal/mst/f_distal_mstXL.dae"
+          </xacro:if>
+          <xacro:if value="${tip_sensor == 'bt_sp'}">
+            <mesh filename="package://sr_description/meshes/components/f_distal/bt_sp/f_distal_bt_sp.dae"
                   scale="0.001 0.001 0.001" />
-            </xacro:if>
-          </geometry>
-        </collision>
+          </xacro:if>
+          <xacro:if value="${tip_sensor == 'bt_2p'}">
+            <mesh filename="package://sr_description/meshes/components/f_distal/bt_2p/f_distal_bt_2p.dae" />
+          </xacro:if>
+          <xacro:if value="${tip_sensor == 'mst'}">
+            <mesh filename="package://sr_description/meshes/components/f_distal/mst/f_distal_mstXL.dae"
+                scale="0.001 0.001 0.001" />
+          </xacro:if>
+        </geometry>
+      </visual>
+      <collision>
+        <origin xyz="0 0 0" rpy="0 0 0" />
+        <geometry name="${prefix}${link_prefix}distal_collision_geom">
+          <xacro:if value="${tip_sensor == 'pst'}">
+            <mesh filename="package://sr_description/meshes/components/f_distal/pst/f_distal_pst.dae"
+                  scale="0.001 0.001 0.001" />
+          </xacro:if>
+          <xacro:if value="${tip_sensor == 'bt_sp'}">
+            <mesh filename="package://sr_description/meshes/components/f_distal/bt_sp/f_distal_bt_sp.dae"
+                  scale="0.001 0.001 0.001" />
+          </xacro:if>
+          <xacro:if value="${tip_sensor == 'bt_2p'}">
+            <mesh filename="package://sr_description/meshes/components/f_distal/bt_2p/f_distal_bt_2p.dae" />
+          </xacro:if>
+          <xacro:if value="${tip_sensor == 'mst'}">
+            <mesh filename="package://sr_description/meshes/components/f_distal/mst/f_distal_mstXL.dae"
+                scale="0.001 0.001 0.001" />
+          </xacro:if>
+        </geometry>
+      </collision>
     </link>
     <xacro:unless value="${tip_sensor == 'bt_2p'}">

Commit message: Update MST meshes (and xacro) to MSTXL and adding MST sensors taxels TFs to the Hand TF tree. (#168)
* Fixing dae files

* Adding finger distal mst

* Fixing finger distal mst

* Adding thumb distal mst

* Adding thumb distal mst

* Adding colour to the thumb mst

* Playing with colours

* Playing with colours

* Changing path

* Adding meshes

* Fixing lint

* wip

* Currently working with the wrong mesh and taxel tfs positions

* Update hand tf tree to include correct mst tfs

* Add thumb new_sensor tfs

* Update MST meshes (and xacro) to MSTXL

* Fix identation

* Update license year

* adding mst xacros, meshes

* undo formatting commit

* formatting

* licence types

* update licence years

* missed a few sr_mst refs

* add comment to explain why mst is treated differently

---------

Co-authored-by: Beatriz Leon <beatriz@shadowrobot.com>
Co-authored-by: carebare47 <tom@shadowrobot.com>
Co-authored-by: Tom Queen <tom_q@hotmail.co.uk>

File: sr_description/hand/xacro/finger/distal/distal.urdf.xacro (robot description, xacro)
@@ -2,5 +2,5 @@
 <!--
  Software License Agreement (BSD License)
- Copyright © 2022 belongs to Shadow Robot Company Ltd.
+ Copyright © 2022-2024 belongs to Shadow Robot Company Ltd.
  All rights reserved.
  Redistribution and use in source and binary forms, with or without modification,
@@ -33,4 +33,5 @@
   <xacro:include filename="$(find sr_description)/hand/xacro/finger/distal/distal.gazebo.xacro" />
   <xacro:include filename="$(find sr_description)/hand/xacro/finger/distal/distal.transmission.xacro" />
+  <xacro:include filename="$(find sr_description)/hand/xacro/finger/distal/f_distal_mstXL.urdf.xacro" />
   <xacro:macro name="distal" params="prefix:=^ link_prefix:=^ joint_prefix:=^ tip_sensor:=^|pst parent">
     <link name="${prefix}${link_prefix}distal">
@@ -54,4 +55,8 @@
             <mesh filename="package://sr_description/meshes/components/f_distal/bt_2p/f_distal_bt_2p.dae" />
           </xacro:if>
+          <xacro:if value="${tip_sensor == 'mst'}">
+            <mesh filename="package://sr_description/meshes/components/f_distal/mst/f_distal_mstXL.dae"
+                scale="0.001 0.001 0.001" />
+          </xacro:if>
         </geometry>
       </visual>
@@ -69,4 +74,8 @@
           <xacro:if value="${tip_sensor == 'bt_2p'}">
             <mesh filename="package://sr_description/meshes/components/f_distal/bt_2p/f_distal_bt_2p.dae" />
+          </xacro:if>
+          <xacro:if value="${tip_sensor == 'mst'}">
+            <mesh filename="package://sr_description/meshes/components/f_distal/mst/f_distal_mstXL.dae"
+                scale="0.001 0.001 0.001" />
           </xacro:if>
         </geometry>
@@ -98,4 +107,8 @@
         <origin xyz="0 0 0.026" rpy="0 0 0" />
       </joint>
+      <!-- For mst we add a link for every taxel in the sensor -->
+      <xacro:if value="${tip_sensor == 'mst'}">
+        <xacro:f_mstXL_distal prefix="${prefix}" link_prefix="${link_prefix}" parent="${prefix}${link_prefix}distal" scale="0.001" show_mesh="false"/>
+      </xacro:if>
     </xacro:unless>
     <!-- extensions -->

File: sr_description/hand/xacro/process_sensor_parameters.xacro (robot description, xacro)
@@ -2,5 +2,5 @@
 <!--
  Software License Agreement (BSD License)
- Copyright © 2022 belongs to Shadow Robot Company Ltd.
+ Copyright © 2022-2024 belongs to Shadow Robot Company Ltd.
  All rights reserved.
  Redistribution and use in source and binary forms, with or without modification,
@@ -59,5 +59,5 @@
 	<xacro:macro name="transform_to_type" params="name value default_tactile_sensor:=^|none
 				valid_finger_tokens:=^|${'th ff mf rf lf'.split()}
-				valid_sensor_tokens:=^|${'bt_2p bt_sp pst none'.split()}">
+				valid_sensor_tokens:=^|${'bt_2p bt_sp pst mst none'.split()}">
 		<!-- None acts as marker indicating that we didn't find the correct type specifier yet -->
 		<!-- Finally, _tmp_ should become a list of (finger, sensor) pairs -->

File: sr_description/hand/xacro/thumb/thdistal.urdf.xacro (robot description, xacro)
@@ -2,5 +2,5 @@
 <!--
  Software License Agreement (BSD License)
- Copyright © 2022, 2023 belongs to Shadow Robot Company Ltd.
+ Copyright © 2022-2024 belongs to Shadow Robot Company Ltd.
  All rights reserved.
  Redistribution and use in source and binary forms, with or without modification,
@@ -33,4 +33,5 @@
   <xacro:include filename="$(find sr_description)/hand/xacro/thumb/thdistal.gazebo.xacro" />
   <xacro:include filename="$(find sr_description)/hand/xacro/thumb/thdistal.transmission.xacro" />
+  <xacro:include filename="$(find sr_description)/hand/xacro/thumb/th_distal_mst.urdf.xacro" />
   <xacro:macro name="thdistal" params="tip_sensor:=^|pst prefix:=^ parent">
     <xacro:if value="${tip_sensor == 'bt_2p'}">
@@ -132,4 +133,8 @@
                     scale="0.001 0.001 0.001" />
             </xacro:if>
+            <xacro:if value="${tip_sensor == 'mst'}">
+              <mesh filename="package://sr_description/meshes/components/th_distal/mst/th_distal_mst.dae"
+                    scale="0.001 0.001 0.001" />
+            </xacro:if>
             <xacro:if value="${tip_sensor == 'bt_sp'}">
               <mesh filename="package://sr_description/meshes/components/th_distal/bt_sp/th_distal_bt_sp.dae"
@@ -150,4 +155,8 @@
             <xacro:if value="${tip_sensor == 'pst'}">
               <mesh filename="package://sr_description/meshes/components/th_distal/pst/th_distal_pst.dae"
+                    scale="0.001 0.001 0.001" />
+            </xacro:if>
+            <xacro:if value="${tip_sensor == 'mst'}">
+              <mesh filename="package://sr_description/meshes/components/th_distal/mst/th_distal_mst.dae"
                     scale="0.001 0.001 0.001" />
             </xacro:if>
@@ -186,4 +195,7 @@
         <origin xyz="0 0 0.0275" rpy="0 0 0" />
       </joint>
+      <xacro:if value="${tip_sensor == 'mst'}">
+        <xacro:t_mst_distal prefix="${prefix}" link_prefix="th" parent="${prefix}thdistal" scale="0.001" show_mesh="false"/>
+      </xacro:if>
       <xacro:thdistal_gazebo />
     </xacro:unless>
