Commit message: Fix thj2 offset in bt_2p configuration
This is an 11 year old fixme that simply asked to remove an arbitrary constant that broke the model.
The links are centered on the joint axis already just as with the other configurations.

We just found that through a lot of manual calibration work..

File: sr_description/hand/xacro/thumb/thmiddle.urdf.xacro (robot description, xacro)
@@ -91,11 +91,5 @@
       <parent link="${parent}" />
       <child link="${prefix}thmiddle" />
-      <xacro:if value="${mid_sensor == 'bt_2p'}">
-        <origin xyz="0 0 0.01" rpy="0 0 0" />
-        <!-- FIXME: z offset is too large -->
-      </xacro:if>
-      <xacro:unless value="${mid_sensor == 'bt_2p'}">
-        <origin xyz="0 0 0" rpy="0 0 0" />
-      </xacro:unless>
+      <origin xyz="0 0 0" rpy="0 0 0" />
       <axis xyz="1 0 0" />
       <limit lower="${-40/180*pi}" upper="${40/180*pi}" effort="2.0" velocity="2.0" />

Commit message: Fix thj2 offset in bt_2p configuration (#171)
* Fix thj2 offset in bt_2p configuration
The links are already centred on the joint axis, just as with the other configurations.

---------

Co-authored-by: devops-shadowrobot <33877923+devops-shadowrobot@users.noreply.github.com>
Co-authored-by: dg-shadow <dg@shadowrobot.com>

File: sr_description/hand/xacro/thumb/thmiddle.urdf.xacro (robot description, xacro)
@@ -2,5 +2,5 @@
 <!--
  Software License Agreement (BSD License)
- Copyright © 2022-2023 belongs to Shadow Robot Company Ltd.
+ Copyright © 2022-2024 belongs to Shadow Robot Company Ltd.
  All rights reserved.
  Redistribution and use in source and binary forms, with or without modification,
@@ -91,11 +91,5 @@
       <parent link="${parent}" />
       <child link="${prefix}thmiddle" />
-      <xacro:if value="${mid_sensor == 'bt_2p'}">
-        <origin xyz="0 0 0.01" rpy="0 0 0" />
-        <!-- FIXME: z offset is too large -->
-      </xacro:if>
-      <xacro:unless value="${mid_sensor == 'bt_2p'}">
-        <origin xyz="0 0 0" rpy="0 0 0" />
-      </xacro:unless>
+      <origin xyz="0 0 0" rpy="0 0 0" />
       <axis xyz="1 0 0" />
       <limit lower="${-40/180*pi}" upper="${40/180*pi}" effort="2.0" velocity="2.0" />
