Commit message: Update colors of FF, MF, RF, and LF STF (MST) distals, from white to black (thumb was already black). Add resources necessary to make the new palm compatible with hand E lite

File: sr_description/hand/xacro/process_hand_type_version_side_parameters.xacro (robot description, xacro)
@@ -27,5 +27,5 @@
 	<xacro:include filename="$(find sr_description)/hand/xacro/validate_macros.xacro" />
 	<xacro:property name="allowed_hand_types" value="${python.set('hand_e hand_g hand_c'.split())}" />
-	<xacro:property name="allowed_hand_versions" value="${python.set('E4 E3M5 E2M3 C6M2 G1M5'.split())}"/>
+	<xacro:property name="allowed_hand_versions" value="${python.set('E4 E3M5 E2M3 C6M2 G4 G1M5'.split())}"/>
         <xacro:property name="allowed_sides" value="${python.set('right left'.split())}"/>
         <xacro:property name="allowed_mounting_plate" value="${python.set([False, True])}"/>

Commit message: New hand G (lite) version with new plam flesh - Hand version G4 (#172)
* Update colors of FF, MF, RF, and LF STF (MST) distals, from white to black (thumb was already black). Add resources necessary to make the new palm compatible with hand E lite

* Other fixes

* Update license years

* Fix weird spacing issue?

* Fix identation

* More identation fixing

---------

Co-authored-by: rnzenha-s <rodrigo@shadowrobot.com>

File: sr_description/hand/xacro/process_hand_type_version_side_parameters.xacro (robot description, xacro)
@@ -2,5 +2,5 @@
 <!--
  Software License Agreement (BSD License)
- Copyright © 2022-2023 belongs to Shadow Robot Company Ltd.
+ Copyright © 2022-2024 belongs to Shadow Robot Company Ltd.
  All rights reserved.
  Redistribution and use in source and binary forms, with or without modification,
@@ -27,5 +27,5 @@
 	<xacro:include filename="$(find sr_description)/hand/xacro/validate_macros.xacro" />
 	<xacro:property name="allowed_hand_types" value="${python.set('hand_e hand_g hand_c'.split())}" />
-	<xacro:property name="allowed_hand_versions" value="${python.set('E4 E3M5 E2M3 C6M2 G1M5'.split())}"/>
+	<xacro:property name="allowed_hand_versions" value="${python.set('E4 E3M5 E2M3 C6M2 G4 G1M5'.split())}"/>
         <xacro:property name="allowed_sides" value="${python.set('right left'.split())}"/>
         <xacro:property name="allowed_mounting_plate" value="${python.set([False, True])}"/>

File: sr_description/robots/sr_hand_bimanual.urdf.xacro (robot description, xacro)
@@ -1,5 +1,5 @@
 <!--
  Software License Agreement (BSD License)
- Copyright © 2022 belongs to Shadow Robot Company Ltd.
+ Copyright © 2022, 2024 belongs to Shadow Robot Company Ltd.
  All rights reserved.
  Redistribution and use in source and binary forms, with or without modification,
@@ -33,5 +33,5 @@
   <xacro:arg name="arm_x_separation" default="-0.4"/>
   <xacro:arg name="right_hand_type" default="hand_e"/>
-  <xacro:arg name="right_hand_version" default="E3M5"/>
+  <xacro:arg name="right_hand_version" default="E4"/>
   <xacro:arg name="right_fingers" default="all"/>
   <xacro:arg name="right_tip_sensors" default="pst"/>
@@ -41,5 +41,5 @@
   <xacro:arg name="right_mounting_plate" default="false"/>
   <xacro:arg name="left_hand_type" default="hand_e"/>
-  <xacro:arg name="left_hand_version" default="E3M5"/>
+  <xacro:arg name="left_hand_version" default="E4"/>
   <xacro:arg name="left_fingers" default="all"/>
   <xacro:arg name="left_tip_sensors" default="pst"/>
